Commit message: commit vecchio urdf

File: urdf/robot_nav2.xacro (robot description, xacro)
@@ -55,4 +55,5 @@
     <!-- pose and inertial -->
     <pose>0 0 0.1 0 0 0</pose>
+    <!-- removed inertia
     <inertial>
       <mass value="5"/>
@@ -60,4 +61,5 @@
       <inertia ixx="0.0395416666667" ixy="0" ixz="0" iyy="0.106208333333" iyz="0" izz="0.106208333333"/>
     </inertial>
+    -->
     <!-- body -->
     <collision name="collision_chassis">
@@ -117,5 +119,5 @@
   <joint name="camera_joint" type="fixed">
     <axis xyz="0 1 0"/>
-    <origin xyz="0.23 0 0.0 " rpy="0 0 0"/>
+    <origin xyz="0.23 0 0.05 " rpy="0 0 0"/>
     <parent link="link_chassis"/>
     <child link="camera_link"/>

Commit message: comunque non funziona

File: urdf/robot_nav2.xacro (robot description, xacro)
@@ -2,58 +2,45 @@
 <robot xmlns:xacro="http://www.ros.org/wiki/xacro" name="robot_nav2_xacro">
  <xacro:include filename="$(find rob_nav2)/urdf/robot_nav2.gazebo"/>
- <xacro:include filename="$(find rob_nav2)/urdf/materials.xacro" />
-  <!-- Inertia definition (cylinder, wheel + chassis) -->
-  <xacro:macro name="cylinder_inertia" params="mass r l">
-    <inertia ixx="${mass*(3*r*r+l*l)/12}" ixy = "0" ixz = "0"
-                iyy="${mass*(3*r*r+l*l)/12}" iyz = "0" izz="${mass*(r*r)/2}" />
-  </xacro:macro>
+	<xacro:property name="length_wheel" value="0.04" />
+	<xacro:property name="radius_wheel" value="0.1" />
 	<xacro:macro name="default_inertial" params="mass">
-      <inertial>
-        <mass value="${mass}" />
-        <origin rpy="0 1.5707 1.5707" xyz="0 0 0"/>
-        <inertia ixx="0.000526666666667" ixy="0" ixz="0" iyy="0.000526666666667" iyz="0" izz="0.001"/>
-      </inertial>
+               <inertial>
+                       <mass value="${mass}" />
+                       <origin rpy="0 1.5707 1.5707" xyz="0 0 0"/>
+                       <inertia ixx="0.000526666666667" ixy="0" ixz="0" iyy="0.000526666666667" iyz="0" izz="0.001"/>
+               </inertial>
 	</xacro:macro>
-  <!-- Wheel defnition -->
-  <xacro:property name="length_wheel" value="0.04" />
-	<xacro:property name="radius_wheel" value="0.1" />
-  <xacro:property name="mass_wheel" value="0.2" />
-  <!-- geometry-->
-  <xacro:macro name="wheel_geometry">
+    <xacro:macro name="wheel_geometry">
 		<geometry>
        			<cylinder length="${length_wheel}" radius="${radius_wheel}"/>
      	</geometry>
 	</xacro:macro>
-  <!-- link -->
-  <xacro:macro name="link_wheel" params="name">
-    <link name="${name}">
-        <xacro:default_inertial mass="${mass_wheel}"/>
-        <collision name="${name}_collision">
-          <origin rpy="0 1.5707 1.5707" xyz="0 0 0"/>
-          <xacro:wheel_geometry />
-        </collision>
-        <visual name="${name}_visual">
-          <origin rpy="0 1.5707 1.5707" xyz="0 0 0"/>
-          <xacro:wheel_geometry />
-          <material name="red"/>
-        </visual>
-    </link>
-  </xacro:macro>
-  <!-- joint -->
-  <xacro:macro name="joint_wheel" params="name child origin_xyz">
-    <joint name="${name}" type="continuous">
-      <origin rpy="0 0 0" xyz="${origin_xyz}"/>
-      <child link="${child}"/>
-      <parent link="link_chassis"/>
-      <axis rpy="0 0 0" xyz="0 1 0"/>
-      <limit effort="10000" velocity="1000"/>
-      <joint_properties damping="1.0" friction="1.0"/>
-    </joint>
-  </xacro:macro>
-  <!-- Chassis definition -->
-  <link name="link_chassis">
+  <material name="black">
+    <color rgba="0.0 0.0 0.0 1.0"/>
+  </material>
+  <material name="blue">
+    <color rgba="0.203125 0.23828125 0.28515625 1.0"/>
+  </material>
+  <material name="green">
+    <color rgba="0.0 0.8 0.0 1.0"/>
+  </material>
+  <material name="grey">
+    <color rgba="0.2 0.2 0.2 1.0"/>
+  </material>
+  <material name="orange">
+    <color rgba="1.0 0.423529411765 0.0392156862745 1.0"/>
+  </material>
+  <material name="brown">
+    <color rgba="0.870588235294 0.811764705882 0.764705882353 1.0"/>
+  </material>
+  <material name="red">
+    <color rgba="0.80078125 0.12890625 0.1328125 1.0"/>
+  </material>
+  <material name="white">
+    <color rgba="1.0 1.0 1.0 1.0"/>
+  </material>
+	  <link name="link_chassis">
     <!-- pose and inertial -->
     <pose>0 0 0.1 0 0 0</pose>
-    <!-- removed inertia
     <inertial>
       <mass value="5"/>
@@ -61,5 +48,4 @@
       <inertia ixx="0.0395416666667" ixy="0" ixz="0" iyy="0.106208333333" iyz="0" izz="0.106208333333"/>
     </inertial>
-    -->
     <!-- body -->
     <collision name="collision_chassis">
@@ -89,37 +75,71 @@
     </visual>
   </link>
-  <!-- Wheel Creation -->
-  <xacro:link_wheel name="link_right_wheel" />
-  <xacro:link_wheel name="link_left_wheel" />
-  <xacro:joint_wheel name="joint_right_wheel"  child="link_right_wheel"  origin_xyz="-0.05 0.15 0"  />
-  <xacro:joint_wheel name="joint_left_wheel"   child="link_left_wheel"   origin_xyz="-0.05 -0.15 0"  />
-  <!-- Camera -->
+   <link name="link_right_wheel">
+    <xacro:default_inertial mass="0.2"/>
+    <collision name="link_right_wheel_collision">
+      <origin rpy="0 1.5707 1.5707" xyz="0 0 0"/>
+      <xacro:wheel_geometry />
+    </collision>
+    <visual name="link_right_wheel_visual">
+      <origin rpy="0 1.5707 1.5707" xyz="0 0 0"/>
+      <xacro:wheel_geometry />
+      <material name="red"/>
+    </visual>
+  </link>
+   <link name="link_left_wheel">
+    <xacro:default_inertial mass="0.2"/>
+    <collision name="link_left_wheel_collision">
+      <origin rpy="0 1.5707 1.5707" xyz="0 0 0"/>
+      <xacro:wheel_geometry />
+    </collision>
+    <visual name="link_left_wheel_visual">
+      <origin rpy="0 1.5707 1.5707" xyz="0 0 0"/>
+      <xacro:wheel_geometry />
+      <material name="red"/>
+    </visual>
+  </link>
+  <joint name="joint_right_wheel" type="continuous">
+    <origin rpy="0 0 0" xyz="-0.05 0.15 0"/>
+    <child link="link_right_wheel"/>
+    <parent link="link_chassis"/>
+    <axis rpy="0 0 0" xyz="0 1 0"/>
+    <limit effort="10000" velocity="1000"/>
+    <joint_properties damping="1.0" friction="1.0"/>
+  </joint>
+  <joint name="joint_left_wheel" type="continuous">
+    <origin rpy="0 0 0" xyz="-0.05 -0.15 0"/>
+    <child link="link_left_wheel"/>
+    <parent link="link_chassis"/>
+    <axis rpy="0 0 0" xyz="0 1 0"/>
+    <limit effort="10000" velocity="1000"/>
+    <joint_properties damping="1.0" friction="1.0"/>
+  </joint>
   <link name="camera_link">
-    <collision>
-      <origin xyz="0 0 0.01" rpy="0 0 0"/>
-      <geometry>
-        <box size="0.05 0.05 0.2"/>
-      </geometry>
-    </collision>
-    <visual>
-      <origin xyz="0 0 0.025" rpy="0 0 0"/>
-      <geometry>
-        <box size="0.05 0.05 0.05"/>
-      </geometry>
-      <material name="red">
-        <color rgba="1 0 0 1"/>
-      </material>
-    </visual>
-    <inertial>
-      <mass value="1e-5"/>
-      <origin xyz="0 0 0" rpy="0 0 0"/>
-      <inertia ixx="1e-6" ixy="0" ixz="0" iyy="1e-6" iyz="0" izz="1e-6"/>
-    </inertial>
+	    <collision>
+	      <origin xyz="0 0 0.1" rpy="0 0 0"/>
+	      <geometry>
+		<box size="0.05 0.05 0.2"/>
+	      </geometry>
+	    </collision>
+	    <visual>
+	      <origin xyz="0 0 0.025" rpy="0 0 0"/>
+	      <geometry>
+		<box size="0.05 0.05 0.05"/>
+	      </geometry>
+	      <material name="red">
+		<color rgba="1 0 0 1"/>
+	      </material>
+	    </visual>
+	    <inertial>
+	      <mass value="1e-5" />
+	      <origin xyz="0 0 0" rpy="0 0 0"/>
+	      <inertia ixx="1e-6" ixy="0" ixz="0" iyy="1e-6" iyz="0" izz="1e-6" />
+	    </inertial>
   </link>
   <joint name="camera_joint" type="fixed">
-    <axis xyz="0 1 0"/>
-    <origin xyz="0.23 0 0.05 " rpy="0 0 0"/>
-    <parent link="link_chassis"/>
-    <child link="camera_link"/>
-  </joint>
+	    <axis xyz="0 1 0" />
+	    <origin xyz="0.23 0 0.235" rpy="0 0 0"/>
+	    <parent link="link_chassis"/>
+	    <child link="camera_link"/>
+	 </joint>
 </robot>

Commit message: secondo me funziona

File: urdf/robot_nav2.xacro (robot description, xacro)
@@ -4,4 +4,10 @@
 	<xacro:property name="length_wheel" value="0.04" />
 	<xacro:property name="radius_wheel" value="0.1" />
+  <xacro:property name="x" value="0.0"/>
+  <xacro:property name="y" value="0.0"/>
+  <xacro:property name="z" value="0.1"/>
+  <xacro:property name="roll" value="0.0"/>
+  <xacro:property name="pitch" value="0.0"/>
+  <xacro:property name="yaw" value="0.0"/>
 	<xacro:macro name="default_inertial" params="mass">
                <inertial>
@@ -42,5 +48,5 @@
 	  <link name="link_chassis">
     <!-- pose and inertial -->
-    <pose>0 0 0.1 0 0 0</pose>
+    <pose>{x} ${y} ${z} ${roll} ${pitch} ${yaw}</pose>
     <inertial>
       <mass value="5"/>

Commit message: aggiustando branches

File: urdf/robot_nav2.xacro (robot description, xacro)
@@ -4,10 +4,4 @@
 	<xacro:property name="length_wheel" value="0.04" />
 	<xacro:property name="radius_wheel" value="0.1" />
-  <xacro:property name="x" value="0.0"/>
-  <xacro:property name="y" value="0.0"/>
-  <xacro:property name="z" value="0.1"/>
-  <xacro:property name="roll" value="0.0"/>
-  <xacro:property name="pitch" value="0.0"/>
-  <xacro:property name="yaw" value="0.0"/>
 	<xacro:macro name="default_inertial" params="mass">
                <inertial>
@@ -48,5 +42,5 @@
 	  <link name="link_chassis">
     <!-- pose and inertial -->
-    <pose>{x} ${y} ${z} ${roll} ${pitch} ${yaw}</pose>
+    <pose>0 0 0.1 0 0 0</pose>
     <inertial>
       <mass value="5"/>
@@ -145,5 +139,5 @@
   <joint name="camera_joint" type="fixed">
 	    <axis xyz="0 1 0" />
-	    <origin xyz="0.23 0 0.235" rpy="0 0 0"/>
+	    <origin xyz="0.23 0 0.1" rpy="0 0 0"/>
 	    <parent link="link_chassis"/>
 	    <child link="camera_link"/>
